File: Schematic/Cherry_MX_Keyboard.sch (EAGLE design)
At the start: 40 parts

Commit message: initial commit for the wireless keyboard
Parts:
- removed B1: PRO_MICRO, SparkFun-Boards:SPARKFUN_PRO_MICRO
- added D1: RED, SparkFun-LED:LED-3MM-NO_SILK
- added D2: GREEN, SparkFun-LED:LED-3MM-NO_SILK
- added R21, R22: 330, SparkFun-Resistors:330OHM-0603-1/10W-1%
- added S19: PWR, SparkFun-Switches:MOMENTARY-SWITCH-SPST-PTH-12MM
- added U1: ESP32_Thing_Plus, SparkFun-RF:ESP-WROOM-32
Connections:
- removed net L_SW: B1.4, S17.SW+
- removed net ROW0: B1.A3, R1.1, R2.2, S1.1
- removed net ROW2: B1.A1, R10.2, R9.1, S9.1
- removed net R_SW: B1.*9, S18.SW+
- new net !GRN_LED: R22.1, U1.MISO_H/IO12
- new net !RED_LED: R21.1, U1.IO27
- new net ENCODER_L_SW: S17.SW+, U1.XTAL_P/IO32
- new net ENCODER_R_SW: S18.SW+, U1.MOSI_V/IO23
- new net KEYS0: R1.1, R2.2, S1.1, U1.SENSOR_VP/I36
- new net KEYS1: R10.2, R9.1, S9.1, U1.SENSOR_VN/I39
- new net N$13: D1.C, R21.2
- new net N$14: R12.1, R13.2, S12.1
- new net N$15: D2.C, R22.2
- new net V_BATT: U1.IO34
- net 3.3V: now also D1.A, D2.A, U1.3V3; no longer B1.VCC, R13.2, R5.2
- net ENCODER_L0: now also U1.XTAL_N/IO33; no longer B1.2
- net ENCODER_L1: now also U1.CS0_H/IO15; no longer B1.*3
- net ENCODER_R0: now also U1.SCK_H/IO14; no longer B1.7
- net ENCODER_R1: now also U1.IO22; no longer B1.8
- net GND: now also S19.1, U1.GND; no longer B1.GND@2
- net N$1: now also R5.2
- net N$7: now also S19.2, U1.EN; no longer R12.1, S12.1
- net ROW1: no longer B1.A2
- net ROW3: no longer B1.A0
Other:
- note added: "v2"
- note removed: "v1"
- moved on the sheet: R1, R10, R11, R12, R13, R14, R15, R16, R17, R18, R19, R2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
